File: kicad/bms-c1.kicad_sch (KiCad schematic)
At the start: 34 parts, among them J1 MicroFit 2x12, J2 B4B-PH-SM4, J3 USB_C_Receptacle_USB2.0, J4 B3B-PH-SM4, J5 B2B-PH-SM4, J6 B4B-PH-SM4, P1 CONN_01X01, P2 CONN_01X01, P3 CONN_01X01, P4 CONN_01X01, P5 CONN_01X01

Commit message: power terminals THT, add mask
Parts:
- P1, P2, P3, P4: footprint LibreSolar:Wuerth_PowerOne_SMD_LF990005 -> open-pe:Wuerth_PowerPlus_M5_Nut
Changed lines of the file:
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@@
 			)
 		)
-		(property "Footprint" "LibreSolar:Wuerth_PowerOne_SMD_LF990005"
+		(property "Footprint" "open-pe:Wuerth_PowerPlus_M5_Nut"
 			(at 144.78 55.88 0)
 			(effects
@@
 			)
 		)
-		(property "Footprint" "LibreSolar:Wuerth_PowerOne_SMD_LF990005"
+		(property "Footprint" "open-pe:Wuerth_PowerPlus_M5_Nut"
 			(at 73.66 63.5 0)
 			(effects
@@
 			)
 		)
-		(property "Footprint" "LibreSolar:Wuerth_PowerOne_SMD_LF990005"
+		(property "Footprint" "open-pe:Wuerth_PowerPlus_M5_Nut"
 			(at 144.78 48.26 0)
 			(effects
@@
 			)
 		)
-		(property "Footprint" "LibreSolar:Wuerth_PowerOne_SMD_LF990005"
+		(property "Footprint" "open-pe:Wuerth_PowerPlus_M5_Nut"
 			(at 73.66 48.26 0)
 			(effects
